Commit message: mpe

File: abb_irb120_support/urdf/irb120_3_58_macro.xacro (robot description, xacro)
@@ -411,5 +411,5 @@
     </joint>
     <joint name="${prefix}joint_6_m" type="revolute">
-      <origin rpy="0 -1.0821 0" xyz="-0.302 0 0"/>
+      <origin rpy="0 0 0" xyz="-0.302 0 0"/>
       <parent link="${prefix}link_4_m"/>
       <child link="${prefix}link_5_m"/>

Commit message: acs

File: abb_irb120_support/urdf/irb120_3_58_macro.xacro (robot description, xacro)
@@ -411,5 +411,5 @@
     </joint>
     <joint name="${prefix}joint_6_m" type="revolute">
-      <origin rpy="0 0 0" xyz="-0.302 0 0"/>
+      <origin rpy="0 0 0" xyz="0.302 0 0"/>
       <parent link="${prefix}link_4_m"/>
       <child link="${prefix}link_5_m"/>
@@ -419,5 +419,5 @@
     </joint>
     <joint name="${prefix}joint_7_m" type="revolute">
-      <origin rpy="0 0 0" xyz="-0.072 0 0"/>
+      <origin rpy="0 0 0" xyz="0.072 0 0"/>
       <parent link="${prefix}link_5_m"/>
       <child link="${prefix}link_6_m"/>

Commit message: acs

File: abb_irb120_support/urdf/irb120_3_58_macro.xacro (robot description, xacro)
@@ -407,17 +407,17 @@
       <child link="${prefix}link_4_m"/>
       <limit effort="0" lower="-2.79253" upper="2.79253" velocity="5.58505"/>
-      <axis xyz="1 0 0"/>
+      <axis xyz="-1 0 0"/>
       <dynamics damping="0.0" friction="0.0"/>
     </joint>
     <joint name="${prefix}joint_6_m" type="revolute">
-      <origin rpy="0 0 0" xyz="0.302 0 0"/>
+      <origin rpy="0 0 0" xyz="-0.302 0 0"/>
       <parent link="${prefix}link_4_m"/>
       <child link="${prefix}link_5_m"/>
       <limit effort="0" lower="-2.094395" upper="2.094395" velocity="5.58505"/>
-      <axis xyz="0 1 0"/>
+      <axis xyz="0 -1 0"/>
       <dynamics damping="0.0" friction="0.0"/>
     </joint>
     <joint name="${prefix}joint_7_m" type="revolute">
-      <origin rpy="0 0 0" xyz="0.072 0 0"/>
+      <origin rpy="0 0 0" xyz="-0.072 0 0"/>
       <parent link="${prefix}link_5_m"/>
       <child link="${prefix}link_6_m"/>

Commit message: added the gripper assembly to rob2

File: abb_irb120_support/urdf/irb120_3_58_macro.xacro (robot description, xacro)
@@ -309,4 +309,20 @@
         </geometry>
         <xacro:material_abb_yellow />
+      </collision>
+    </link>
+    <!-- gripper assembly -->
+    <link name="${prefix}gripper_assembly">
+      <visual>
+        <origin xyz="0 0 0" rpy="0 0 0"/>
+        <geometry>
+          <mesh filename="package://abb_irb120_support/meshes/irb120_3_58/visual/gripper_assembly.stl" scale="0.001 0.001 0.001"/>
+        </geometry>
+        <xacro:material_abb_white />
+      </visual>
+      <collision>
+        <origin xyz="0 0 0" rpy="0 0 0"/>
+        <geometry>
+          <mesh filename="package://abb_irb120_support/meshes/irb120_3_58/collision/gripper_collision_cube.stl" scale="0.001 0.001 0.001"/>
+        </geometry>
       </collision>
     </link>
@@ -484,4 +500,9 @@
       <child link="${prefix}tool0_m" />
     </joint>
+    <joint name="${prefix}gripper_joint" type="fixed">
+      <origin rpy="0 ${radians(-90)} 0" xyz="0 0 0"/>
+      <parent link="${prefix}flange_m"/>
+      <child link="${prefix}gripper_assembly"/>
+    </joint>
   </xacro:macro>
 </robot>

Commit message: modified eef position to be in between the gripper figures; added a ground plane

File: abb_irb120_support/urdf/irb120_3_58_macro.xacro (robot description, xacro)
@@ -324,4 +324,20 @@
         <geometry>
           <mesh filename="package://abb_irb120_support/meshes/irb120_3_58/collision/gripper_collision_cube.stl" scale="0.001 0.001 0.001"/>
+        </geometry>
+      </collision>
+    </link>
+    <!-- ground plane -->
+    <link name="${prefix}ground">
+      <visual>
+        <origin xyz="0 0 0" rpy="0 0 0"/>
+        <geometry>
+          <mesh filename="package://abb_irb120_support/meshes/irb120_3_58/visual/ground_plane.stl" scale="0.001 0.001 0.001"/>
+        </geometry>
+        <xacro:material_abb_white />
+      </visual>
+      <collision>
+        <origin xyz="0 0 0" rpy="0 0 0"/>
+        <geometry>
+          <mesh filename="package://abb_irb120_support/meshes/irb120_3_58/collision/ground_plane.stl" scale="0.001 0.001 0.001"/>
         </geometry>
       </collision>
@@ -496,5 +512,5 @@
     <link name="${prefix}tool0_m" />
     <joint name="${prefix}link_7_m-tool0_m" type="fixed">
-      <origin xyz="-0.01 0 0" rpy="0 ${radians(90)} 0" />
+      <origin xyz="-0.16 0 0" rpy="0 ${radians(90)} 0" />
       <parent link="${prefix}flange_m" />
       <child link="${prefix}tool0_m" />
@@ -505,4 +521,9 @@
       <child link="${prefix}gripper_assembly"/>
     </joint>
+    <joint name="${prefix}ground_joint" type="fixed">
+      <origin rpy="${radians(90)} 0 0" xyz="0.5 0 0"/>
+      <parent link="${prefix}base_link"/>
+      <child link="${prefix}ground"/>
+    </joint>
   </xacro:macro>
 </robot>
