Commit message: update urdf s.t. arms are 1.09m apart instead of 1m

File: abb_irb120_support/urdf/irb120_3_58.urdf (robot description, URDF)
Before this commit: robot abb_irb120_3_58, 20 links, 19 joints
Links:
- added link gripper_assembly; collision mesh filename=package://abb_irb120_support/meshes/irb120_3_58/collision/g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 scale=0.001 0.001 0.001; visual mesh filename=package://abb_irb120_support/meshes/irb120_3_58/visual/grip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 scale=0.001 0.001 0.001
- added link ground; collision mesh filename=package://abb_irb120_support/meshes/irb120_3_58/collision/g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 scale=0.001 0.001 0.001; visual mesh filename=package://abb_irb120_support/meshes/irb120_3_58/visual/grou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 scale=0.001 0.001 0.001
Joints:
- removed joint joint_1
- removed joint joint_1_m
- added joint dummy-base_link: type fixed, parent dummy, child base_link, origin xyz=0 0 0 rpy=0 0 0
- added joint dummy-base_link_m: type fixed, parent dummy, child base_link_m, origin xyz=0 0 0 rpy=0 0 0
- added joint gripper_joint: type fixed, parent flange_m, child gripper_assembly, origin xyz=0 0 0 rpy=0 -1.5707963267948966 0
- added joint ground_joint: type fixed, parent base_link, child ground, origin xyz=0.5 0 0 rpy=1.5707963267948966 0 0
- joint joint_2_m: origin xyz=1 0 0 rpy=0 0 0 -> xyz=1.09 0 0 rpy=0 0 0
- joint joint_3_m: axis 0 1 0 -> 0 -1 0
- joint joint_4_m: axis 0 1 0 -> 0 -1 0
- joint joint_5_m: axis 1 0 0 -> -1 0 0
- joint joint_6_m: axis 0 1 0 -> 0 -1 0; origin xyz=0.302 0 0 rpy=0 0 0 -> xyz=-0.302 0 0 rpy=0 0 0
- joint joint_7_m: origin xyz=0.072 0 0 rpy=0 0 0 -> xyz=-0.072 0 0 rpy=0 0 0
- joint link_7-tool0: origin xyz=0 0 0 rpy=0 1.57079632679 0 -> xyz=0 0 0 rpy=0 1.5707963267948966 0
- joint link_7_m-tool0_m: origin xyz=0 0 0 rpy=0 1.57079632679 0 -> xyz=-0.16 0 0 rpy=0 1.5707963267948966 0

File: abb_irb120_support/urdf/irb120_3_58_macro.xacro (robot description, xacro)
@@ -171,5 +171,5 @@
       </inertial>
       <visual>
-        <origin xyz="1 0 0" rpy="0 0 3.14159"/>
+        <origin xyz="1.09 0 0" rpy="0 0 3.14159"/>
         <geometry>
           <mesh filename="package://abb_irb120_support/meshes/irb120_3_58/visual/base_link.stl"/>
@@ -178,5 +178,5 @@
       </visual>
       <collision>
-        <origin xyz="1 0 0" rpy="0 0 3.14159"/>
+        <origin xyz="1.09 0 0" rpy="0 0 3.14159"/>
         <geometry>
           <mesh filename="package://abb_irb120_support/meshes/irb120_3_58/collision/base_link.stl"/>
@@ -411,5 +411,5 @@
     </joint> -->
     <joint name="${prefix}joint_2_m" type="revolute">
-      <origin rpy="0 0 0" xyz="1 0 0"/>
+      <origin rpy="0 0 0" xyz="1.09 0 0"/>
       <parent link="${prefix}base_link_m"/>
       <child link="${prefix}link_1_m"/>

Commit message: [WIP] rename dummy link to world link, rm visual element for virtual world link (eliminates 'failed to parse visual element for link 'dummy'' error on dual_arm launch)

File: abb_irb120_support/urdf/irb120_3_58.urdf (robot description, URDF)
Before this commit: robot abb_irb120_3_58, 22 links, 21 joints
Links:
- removed link dummy
- added link world
Joints:
- removed joint dummy-base
- removed joint dummy-base_link
- removed joint dummy-base_link_m
- added joint world-base: type fixed, parent world, child base, origin xyz=0 0 0 rpy=0 0 0
- added joint world-base_link: type fixed, parent world, child base_link, origin xyz=0 0 0 rpy=0 0 0
- added joint world-base_link_m: type fixed, parent world, child base_link_m, origin xyz=0 0 0 rpy=0 0 0

File: abb_irb120_support/urdf/irb120_3_58_macro.xacro (robot description, xacro)
@@ -4,15 +4,6 @@
   <xacro:macro name="abb_irb120_3_58" params="prefix">
     <!-- link list -->
-    <link name="${prefix}dummy">
-      <visual>
+    <link name="${prefix}world">
         <origin xyz="0.5 0 0" rpy="0 0 0"/>
-      </visual>
-      <!--<collision>
-        <origin xyz="0.5 0 0" rpy="0 0 0"/>
-        <geometry>
-          <mesh filename="package://abb_irb120_support/meshes/irb120_3_58/collision/base_link.stl"/>
-        </geometry>
-        <xacro:material_abb_yellow />
-      </collision> -->
     </link>
     <link name="${prefix}base_link">
@@ -347,5 +338,5 @@
     <joint name="${prefix}joint_1" type="revolute">
       <origin rpy="0 0 0" xyz="0.5 0 0"/>
-      <parent link="${prefix}dummy"/>
+      <parent link="${prefix}world"/>
       <child link="${prefix}base_link"/>
       <limit effort="0" lower="-2.87979" upper="2.87979" velocity="4.36332"/>
@@ -404,5 +395,5 @@
     <joint name="${prefix}joint_1_m" type="revolute">
       <origin rpy="0 0 0" xyz="1.5 0 0"/>
-      <parent link="${prefix}dummy"/>
+      <parent link="${prefix}world"/>
       <child link="${prefix}base_link_m"/>
       <limit effort="0" lower="-2.87979" upper="2.87979" velocity="4.36332"/>
@@ -461,31 +452,19 @@
     <!-- ROS-Industrial 'base' frame: base_link to ABB World Coordinates transform -->
     <link name="${prefix}base" />
-    <joint name="${prefix}dummy-base" type="fixed">
+    <joint name="${prefix}world-base" type="fixed">
       <origin xyz="0 0 0" rpy="0 0 0"/>
-      <parent link="${prefix}dummy"/>
+      <parent link="${prefix}world"/>
       <child link="${prefix}base"/>
     </joint>
-    <joint name="${prefix}dummy-base_link" type="fixed">
+    <joint name="${prefix}world-base_link" type="fixed">
       <origin xyz="0 0 0" rpy="0 0 0"/>
-      <parent link="${prefix}dummy"/>
+      <parent link="${prefix}world"/>
       <child link="${prefix}base_link"/>
     </joint>
-    <joint name="${prefix}dummy-base_link_m" type="fixed">
+    <joint name="${prefix}world-base_link_m" type="fixed">
       <origin xyz="0 0 0" rpy="0 0 0"/>
-      <parent link="${prefix}dummy"/>
+      <parent link="${prefix}world"/>
       <child link="${prefix}base_link_m"/>
     </joint>
-    <!--<link name="${prefix}base_1" />
-    <joint name="${prefix}base_link-base" type="fixed">
-      <origin xyz="0 0 0" rpy="0 0 0"/>
-      <parent link="${prefix}base"/>
-      <child link="${prefix}base_link"/>
-    </joint>
-    <link name="${prefix}base_m" />
-    <joint name="${prefix}base_link-base" type="fixed">
-      <origin xyz="0 0 0" rpy="0 0 0"/>
-      <parent link="${prefix}base"/>
-      <child link="${prefix}base_link_m"/>
-    </joint> -->
     <!-- ROS-Industrial 'flange' frame: attachment point for EEF models -->
     <link name="${prefix}flange"/>

Commit message: [WIP] rm unused base virtual joint and link

File: abb_irb120_support/urdf/irb120_3_58.urdf (robot description, URDF)
Before this commit: robot abb_irb120_3_58, 22 links, 21 joints
Links:
- removed link base
Joints:
- removed joint world-base
- joint gripper_joint: origin xyz=0 0 0 rpy=0 -1.5707963267948966 0 -> xyz=0 0 0 rpy=0 ${radians(-90)} 0
- joint ground_joint: origin xyz=0.5 0 0 rpy=1.5707963267948966 0 0 -> xyz=0.5 0 0 rpy=${radians(90)} 0 0
- joint link_7-tool0: origin xyz=0 0 0 rpy=0 1.5707963267948966 0 -> xyz=0 0 0 rpy=0 ${radians(90)} 0
- joint link_7_m-tool0_m: origin xyz=-0.16 0 0 rpy=0 1.5707963267948966 0 -> xyz=0 0 0 rpy=0 ${radians(90)} 0

File: abb_irb120_support/urdf/irb120_3_58_macro.xacro (robot description, xacro)
@@ -335,13 +335,5 @@
     </link>
     <!-- end of link list -->
-    <!-- joint list
-    <joint name="${prefix}joint_1" type="revolute">
-      <origin rpy="0 0 0" xyz="0.5 0 0"/>
-      <parent link="${prefix}world"/>
-      <child link="${prefix}base_link"/>
-      <limit effort="0" lower="-2.87979" upper="2.87979" velocity="4.36332"/>
-      <axis xyz="0 0 1"/>
-      <dynamics damping="0.0" friction="0.0"/>
-    </joint> -->
+    <!-- joint list -->
     <joint name="${prefix}joint_2" type="revolute">
       <origin rpy="0 0 0" xyz="0 0 0"/>
@@ -392,13 +384,4 @@
       <dynamics damping="0.0" friction="0.0"/>
     </joint>
-    <!-- joint list - mirror
-    <joint name="${prefix}joint_1_m" type="revolute">
-      <origin rpy="0 0 0" xyz="1.5 0 0"/>
-      <parent link="${prefix}world"/>
-      <child link="${prefix}base_link_m"/>
-      <limit effort="0" lower="-2.87979" upper="2.87979" velocity="4.36332"/>
-      <axis xyz="0 0 1"/>
-      <dynamics damping="0.0" friction="0.0"/>
-    </joint> -->
     <joint name="${prefix}joint_2_m" type="revolute">
       <origin rpy="0 0 0" xyz="1.09 0 0"/>
@@ -450,11 +433,5 @@
     </joint>
     <!-- end of joint list -->
-    <!-- ROS-Industrial 'base' frame: base_link to ABB World Coordinates transform -->
-    <link name="${prefix}base" />
-    <joint name="${prefix}world-base" type="fixed">
-      <origin xyz="0 0 0" rpy="0 0 0"/>
-      <parent link="${prefix}world"/>
-      <child link="${prefix}base"/>
-    </joint>
+    <!-- ROS-Industrial: base_link to ABB World Coordinates transform -->
     <joint name="${prefix}world-base_link" type="fixed">
       <origin xyz="0 0 0" rpy="0 0 0"/>
@@ -474,5 +451,4 @@
       <child link="${prefix}flange"/>
     </joint>
-    <!-- mirror -->
     <link name="${prefix}flange_m"/>
     <joint type="fixed" name="${prefix}joint_8_m-flange_m">
@@ -488,8 +464,7 @@
       <child link="${prefix}tool0" />
     </joint>
-    <!-- mirror -->
     <link name="${prefix}tool0_m" />
     <joint name="${prefix}link_7_m-tool0_m" type="fixed">
-      <origin xyz="-0.16 0 0" rpy="0 ${radians(90)} 0" />
+      <origin xyz="0 0 0" rpy="0 ${radians(90)} 0" />
       <parent link="${prefix}flange_m" />
       <child link="${prefix}tool0_m" />
