Commit message: [FIX] revert how angles are specified in dual_arm.urdf, test check_urdf.launch

File: abb_irb120_support/urdf/dual_arm.urdf (robot description, URDF)
Before this commit: robot dual_arm, 21 links, 20 joints
Joints:
- joint gripper_joint: origin xyz=0 0 0 rpy=0 ${radians(-90)} 0 -> xyz=0 0 0 rpy=0 -1.5708 0
- joint ground_joint: origin xyz=0.5 0 0 rpy=${radians(90)} 0 0 -> xyz=0.5 0 0 rpy=1.5708 0 0
- joint link_7-tool0: origin xyz=0 0 0 rpy=0 ${radians(90)} 0 -> xyz=0 0 0 rpy=0 1.5708 0
- joint link_7_m-tool0_m: origin xyz=0 0 0 rpy=0 ${radians(90)} 0 -> xyz=0 0 0 rpy=0 1.5708 0

Commit message: finish simplifying frame/tree structure connecting gripper to mp_m in URDF and SRDF files

File: abb_irb120_support/urdf/dual_arm.urdf (robot description, URDF)
Before this commit: robot dual_arm, 21 links, 20 joints
Links:
- removed link flange
- removed link flange_m
- removed link gripper_assembly
- removed link tool0
- removed link tool0_m
- added link gripper_m; collision mesh filename=package://abb_irb120_support/meshes/irb120_3_58/collision/g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 scale=0.001 0.001 0.001; visual mesh filename=package://abb_irb120_support/meshes/irb120_3_58/visual/grip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 scale=0.001 0.001 0.001
Joints:
- removed joint gripper_joint
- removed joint joint_8-flange
- removed joint joint_8_m-flange_m
- removed joint link_7-tool0
- removed joint link_7_m-tool0_m
- added joint gripper_joint_m: type fixed, parent link_6_m, child gripper_m, origin xyz=0 0 0 rpy=0 -1.5708 0

File: abb_irb120_support/urdf/dual_arm_macro.xacro (robot description, xacro)
@@ -302,6 +302,6 @@
       </collision>
     </link>
-    <!-- gripper assembly -->
-    <link name="${prefix}gripper_assembly">
+    <!-- gripper -->
+    <link name="${prefix}gripper_m">
       <visual>
         <origin xyz="0 0 0" rpy="0 0 0"/>
@@ -444,34 +444,8 @@
       <child link="${prefix}base_link_m"/>
     </joint>
-    <!-- ROS-Industrial 'flange' frame: attachment point for EEF models -->
-    <link name="${prefix}flange"/>
-    <joint type="fixed" name="${prefix}joint_8-flange">
-      <origin xyz="0 0 0" rpy="0 0 0"/>
-      <parent link="${prefix}link_6"/>
-      <child link="${prefix}flange"/>
-    </joint>
-    <link name="${prefix}flange_m"/>
-    <joint type="fixed" name="${prefix}joint_8_m-flange_m">
-      <origin xyz="0 0 0" rpy="0 0 0"/>
+    <joint name="${prefix}gripper_joint_m" type="fixed">
+      <origin rpy="0 ${radians(-90)} 0" xyz="0 0 0"/>
       <parent link="${prefix}link_6_m"/>
-      <child link="${prefix}flange_m"/>
-    </joint>
-    <!-- ROS-Industrial 'tool0' frame: all-zeros tool frame -->
-    <link name="${prefix}tool0" />
-    <joint name="${prefix}link_7-tool0" type="fixed">
-      <origin xyz="0 0 0" rpy="0 ${radians(90)} 0" />
-      <parent link="${prefix}flange" />
-      <child link="${prefix}tool0" />
-    </joint>
-    <link name="${prefix}tool0_m" />
-    <joint name="${prefix}link_7_m-tool0_m" type="fixed">
-      <origin xyz="0 0 0" rpy="0 ${radians(90)} 0" />
-      <parent link="${prefix}flange_m" />
-      <child link="${prefix}tool0_m" />
-    </joint>
-    <joint name="${prefix}gripper_joint" type="fixed">
-      <origin rpy="0 ${radians(-90)} 0" xyz="0 0 0"/>
-      <parent link="${prefix}flange_m"/>
-      <child link="${prefix}gripper_assembly"/>
+      <child link="${prefix}gripper_m"/>
     </joint>
     <joint name="${prefix}ground_joint" type="fixed">

Commit message: [DOCS] Simplify frame structure of dual_arm scene and update docs

File: abb_irb120_support/urdf/dual_arm.urdf (robot description, URDF)
Before this commit: robot dual_arm, 17 links, 16 joints
Joints:
- joint ground_joint: parent base_link -> world

File: abb_irb120_support/urdf/dual_arm_macro.xacro (robot description, xacro)
@@ -451,5 +451,5 @@
     <joint name="${prefix}ground_joint" type="fixed">
       <origin rpy="${radians(90)} 0 0" xyz="0.5 0 0"/>
-      <parent link="${prefix}base_link"/>
+      <parent link="${prefix}world"/>
       <child link="${prefix}ground"/>
     </joint>

Commit message: [FIX] Fixed removing unnecessary and redundant frames from dual_arm planning, updated docs, fixed alignment of ground plane .stl file

File: abb_irb120_support/urdf/dual_arm.urdf (robot description, URDF)
Before this commit: robot dual_arm, 17 links, 16 joints
Links:
- removed link ground
- link world: geometry collision mesh filename=package://abb_irb120_support/meshes/irb120_3_58/collision/g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 scale=0.001 0.001 0.001; visual mesh filename=package://abb_irb120_support/meshes/irb120_3_58/visual/grou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 scale=0.001 0.001 0.001
Joints:
- removed joint ground_joint
- joint gripper_joint_m: origin xyz=0 0 0 rpy=0 -1.5708 0 -> xyz=0 0 0 rpy=0 -1.5707963267948966 0
- joint joint_2_m: origin xyz=1.09 0 0 rpy=0 0 0 -> xyz=0 0 0 rpy=0 0 0
- joint world-base_link: origin xyz=0 0 0 rpy=0 0 0 -> xyz=-0.545 0 0 rpy=0 0 0
- joint world-base_link_m: origin xyz=0 0 0 rpy=0 0 0 -> xyz=0.545 0 0 rpy=0 0 0

File: abb_irb120_support/urdf/dual_arm_macro.xacro (robot description, xacro)
@@ -3,8 +3,21 @@
   <xacro:include filename="$(find abb_resources)/urdf/common_materials.xacro"/>
   <xacro:macro name="dual_arm" params="prefix">
-    <!-- link list -->
+    <!-- World Link -->
     <link name="${prefix}world">
-        <origin xyz="0.5 0 0" rpy="0 0 0"/>
-    </link>
+      <visual>
+        <origin xyz="0 0 0" rpy="0 0 0"/>
+        <geometry>
+          <mesh filename="package://abb_irb120_support/meshes/irb120_3_58/visual/ground_plane.stl" scale="0.001 0.001 0.001"/>
+        </geometry>
+        <xacro:material_abb_white />
+      </visual>
+      <collision>
+        <origin xyz="0 0 0" rpy="0 0 0"/>
+        <geometry>
+          <mesh filename="package://abb_irb120_support/meshes/irb120_3_58/collision/ground_plane.stl" scale="0.001 0.001 0.001"/>
+        </geometry>
+      </collision>
+    </link>
+    <!-- Arm 1 Links -->
     <link name="${prefix}base_link">
       <inertial>
@@ -154,6 +167,6 @@
       </collision>
     </link>
-     <!-- mirror for second arm -->
-      <link name="${prefix}base_link_m">
+    <!-- Arm 2 Links -->
+    <link name="${prefix}base_link_m">
       <inertial>
         <mass value="6.215"/>
@@ -162,5 +175,5 @@
       </inertial>
       <visual>
-        <origin xyz="1.09 0 0" rpy="0 0 3.14159"/>
+        <origin xyz="0 0 0" rpy="0 0 3.14159"/>
         <geometry>
           <mesh filename="package://abb_irb120_support/meshes/irb120_3_58/visual/base_link.stl"/>
@@ -169,5 +182,5 @@
       </visual>
       <collision>
-        <origin xyz="1.09 0 0" rpy="0 0 3.14159"/>
+        <origin xyz="0 0 0" rpy="0 0 3.14159"/>
         <geometry>
           <mesh filename="package://abb_irb120_support/meshes/irb120_3_58/collision/base_link.stl"/>
@@ -302,5 +315,5 @@
       </collision>
     </link>
-    <!-- gripper -->
+    <!-- Gripper Links -->
     <link name="${prefix}gripper_m">
       <visual>
@@ -318,22 +331,5 @@
       </collision>
     </link>
-    <!-- ground plane -->
-    <link name="${prefix}ground">
-      <visual>
-        <origin xyz="0 0 0" rpy="0 0 0"/>
-        <geometry>
-          <mesh filename="package://abb_irb120_support/meshes/irb120_3_58/visual/ground_plane.stl" scale="0.001 0.001 0.001"/>
-        </geometry>
-        <xacro:material_abb_white />
-      </visual>
-      <collision>
-        <origin xyz="0 0 0" rpy="0 0 0"/>
-        <geometry>
-          <mesh filename="package://abb_irb120_support/meshes/irb120_3_58/collision/ground_plane.stl" scale="0.001 0.001 0.001"/>
-        </geometry>
-      </collision>
-    </link>
-    <!-- end of link list -->
-    <!-- joint list -->
+    <!-- Arm 1 Joints -->
     <joint name="${prefix}joint_2" type="revolute">
       <origin rpy="0 0 0" xyz="0 0 0"/>
@@ -384,6 +380,7 @@
       <dynamics damping="0.0" friction="0.0"/>
     </joint>
+    <!-- Arm 2 Joints -->
     <joint name="${prefix}joint_2_m" type="revolute">
-      <origin rpy="0 0 0" xyz="1.09 0 0"/>
+      <origin rpy="0 0 0" xyz="0 0 0"/>
       <parent link="${prefix}base_link_m"/>
       <child link="${prefix}link_1_m"/>
@@ -432,16 +429,5 @@
       <dynamics damping="0.0" friction="0.0"/>
     </joint>
-    <!-- end of joint list -->
-    <!-- ROS-Industrial: base_link to ABB World Coordinates transform -->
-    <joint name="${prefix}world-base_link" type="fixed">
-      <origin xyz="0 0 0" rpy="0 0 0"/>
-      <parent link="${prefix}world"/>
-      <child link="${prefix}base_link"/>
-    </joint>
-    <joint name="${prefix}world-base_link_m" type="fixed">
-      <origin xyz="0 0 0" rpy="0 0 0"/>
-      <parent link="${prefix}world"/>
-      <child link="${prefix}base_link_m"/>
-    </joint>
+    <!-- Gripper Joints -->
     <joint name="${prefix}gripper_joint_m" type="fixed">
       <origin rpy="0 ${radians(-90)} 0" xyz="0 0 0"/>
@@ -449,8 +435,14 @@
       <child link="${prefix}gripper_m"/>
     </joint>
-    <joint name="${prefix}ground_joint" type="fixed">
-      <origin rpy="${radians(90)} 0 0" xyz="0.5 0 0"/>
+    <!-- World Joints -->
+    <joint name="${prefix}world-base_link" type="fixed">
+      <origin xyz="-0.545 0 0" rpy="0 0 0"/>
       <parent link="${prefix}world"/>
-      <child link="${prefix}ground"/>
+      <child link="${prefix}base_link"/>
+    </joint>
+    <joint name="${prefix}world-base_link_m" type="fixed">
+      <origin xyz="0.545 0 0" rpy="0 0 0"/>
+      <parent link="${prefix}world"/>
+      <child link="${prefix}base_link_m"/>
     </joint>
   </xacro:macro>

Commit message: [FIX] Update dual_arm.urdf with correct gripper info

File: abb_irb120_support/urdf/dual_arm.urdf (robot description, URDF)
Before this commit: robot dual_arm, 16 links, 15 joints
Joints:
- joint gripper_joint_m: origin xyz=0 0 0 rpy=0 -1.5707963267948966 0 -> xyz=0 0 0 rpy=0 0 0

Commit message: [FIX] add tcp link+joint to URDF, gripper links fully specified. Can plan for gripper tcp in RViz click-and-drag planning+execution.

File: abb_irb120_support/urdf/dual_arm.urdf (robot description, URDF)
Before this commit: robot dual_arm, 16 links, 15 joints
Links:
- added link gripper_base_m
- added link gripper_tcp_m; visual mesh filename=package://abb_irb120_support/meshes/irb120_3_58/visual/cube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 scale=0.0005 0.0005 0.0005
Joints:
- added joint gripper_base_joint_m: type fixed, parent gripper_m, child gripper_base_m, origin xyz=-0.1277 0 0 rpy=0 0 0
- added joint gripper_tcp_joint_m: type fixed, parent gripper_base_m, child gripper_tcp_m, origin xyz=-0.045283 0 0 rpy=-0.3490658503988659 0 0

File: abb_irb120_support/urdf/dual_arm_macro.xacro (robot description, xacro)
@@ -330,4 +330,16 @@
         </geometry>
       </collision>
+    </link>
+    <link name="${prefix}gripper_base_m">
+      <origin xyz="0 0 0" rpy="0 0 0"/>
+    </link>
+    <link name="${prefix}gripper_tcp_m">
+      <visual>
+        <origin xyz="0 0 0" rpy="0 0 0"/>
+        <geometry>
+          <mesh filename="package://abb_irb120_support/meshes/irb120_3_58/visual/cube.stl" scale="0.0005 0.0005 0.0005"/>
+        </geometry>
+        <xacro:material_abb_white />
+      </visual>
     </link>
     <!-- Arm 1 Joints -->
@@ -435,4 +447,15 @@
       <child link="${prefix}gripper_m"/>
     </joint>
+    <joint name="${prefix}gripper_base_joint_m" type="fixed">
+      <origin rpy="0 0 0" xyz="-0.1277 0 0"/>
+      <parent link="${prefix}gripper_m"/>
+      <child link="${prefix}gripper_base_m"/>
+    </joint>
+    <joint name="${prefix}gripper_tcp_joint_m" type="fixed">
+      <!-- <origin rpy="0 0 0" xyz="-0.172 -0.0316545 0.0482436"/> -->
+      <origin rpy="${radians(-20)} 0 0" xyz="-0.045283 0 0"/>
+      <parent link="${prefix}gripper_base_m"/>
+      <child link="${prefix}gripper_tcp_m"/>
+    </joint>
     <!-- World Joints -->
     <joint name="${prefix}world-base_link" type="fixed">
