Commit message: [WIP] rename all dual_arm robot descriptions/controllers from 'abb_irb120_3_58' to 'dual_arm'

File: abb_irb120_support/urdf/dual_arm_macro.xacro (robot description, xacro)
@@ -2,5 +2,5 @@
 <robot xmlns:xacro="http://ros.org/wiki/xacro">
   <xacro:include filename="$(find abb_resources)/urdf/common_materials.xacro"/>
-  <xacro:macro name="abb_irb120_3_58" params="prefix">
+  <xacro:macro name="dual_arm" params="prefix">
     <!-- link list -->
     <link name="${prefix}world">

Commit message: fixed gripper stl orientation

File: abb_irb120_support/urdf/dual_arm_macro.xacro (robot description, xacro)
@@ -431,5 +431,5 @@
     <!-- Gripper Joints -->
     <joint name="${prefix}gripper_joint_m" type="fixed">
-      <origin rpy="0 ${radians(-90)} 0" xyz="0 0 0"/>
+      <origin rpy="0 0 0" xyz="0 0 0"/>
       <parent link="${prefix}link_6_m"/>
       <child link="${prefix}gripper_m"/>

Commit message: [FIX] fix joint axes for mirrored mp_m (all should be -1 for mirroring), fix yaw of all links in mp_m (all should be 180o), remove chains in srdf, fix ee designation in srdf

File: abb_irb120_support/urdf/dual_arm_macro.xacro (robot description, xacro)
@@ -2,5 +2,12 @@
 <robot xmlns:xacro="http://ros.org/wiki/xacro">
   <xacro:include filename="$(find abb_resources)/urdf/common_materials.xacro"/>
-  <xacro:macro name="dual_arm" params="prefix">
+  <xacro:macro name="dual_arm" params="
+  prefix
+  joint_limits_parameters_file:='$(find abb_irb120_moveit_config)/config/joint_limits.yaml'
+  kinematics_parameters_file:='$(find abb_irb120_moveit_config)/config/kinematics.yaml'
+  safety_limits:=false
+  safety_pos_margin:=0.15
+  safety_k_position:=20"
+  >
     <!-- World Link -->
     <link name="${prefix}world">
@@ -175,5 +182,5 @@
       </inertial>
       <visual>
-        <origin xyz="0 0 0" rpy="0 0 3.14159"/>
+        <origin xyz="0 0 0" rpy="0 0 ${radians(180)}"/>
         <geometry>
           <mesh filename="package://abb_irb120_support/meshes/irb120_3_58/visual/base_link.stl"/>
@@ -182,5 +189,5 @@
       </visual>
       <collision>
-        <origin xyz="0 0 0" rpy="0 0 3.14159"/>
+        <origin xyz="0 0 0" rpy="0 0 ${radians(180)}"/>
         <geometry>
           <mesh filename="package://abb_irb120_support/meshes/irb120_3_58/collision/base_link.stl"/>
@@ -196,5 +203,5 @@
       </inertial>
       <visual>
-        <origin xyz="0 0 0" rpy="0 0 3.14159"/>
+        <origin xyz="0 0 0" rpy="0 0 ${radians(180)}"/>
         <geometry>
           <mesh filename="package://abb_irb120_support/meshes/irb120_3_58/visual/link_1.stl"/>
@@ -203,5 +210,5 @@
       </visual>
       <collision>
-        <origin xyz="0 0 0" rpy="0 0 3.14159"/>
+        <origin xyz="0 0 0" rpy="0 0 ${radians(180)}"/>
         <geometry>
           <mesh filename="package://abb_irb120_support/meshes/irb120_3_58/collision/link_1.stl"/>
@@ -217,5 +224,5 @@
       </inertial>
       <visual>
-        <origin xyz="0 0 0" rpy="0 0 0"/>
+        <origin xyz="0 0 0" rpy="0 0 ${radians(180)}"/>
         <geometry>
           <mesh filename="package://abb_irb120_support/meshes/irb120_3_58/visual/link_2.stl"/>
@@ -224,5 +231,5 @@
       </visual>
       <collision>
-        <origin xyz="0 0 0" rpy="0 0 0"/>
+        <origin xyz="0 0 0" rpy="0 0 ${radians(180)}"/>
         <geometry>
           <mesh filename="package://abb_irb120_support/meshes/irb120_3_58/collision/link_2.stl"/>
@@ -238,5 +245,5 @@
       </inertial>
       <visual>
-        <origin xyz="0 0 0" rpy="0 0 3.14159"/>
+        <origin xyz="0 0 0" rpy="0 0 ${radians(180)}"/>
         <geometry>
           <mesh filename="package://abb_irb120_support/meshes/irb120_3_58/visual/link_3.stl"/>
@@ -245,5 +252,5 @@
       </visual>
       <collision>
-        <origin xyz="0 0 0" rpy="0 0 3.14159"/>
+        <origin xyz="0 0 0" rpy="0 0 ${radians(180)}"/>
         <geometry>
           <mesh filename="package://abb_irb120_support/meshes/irb120_3_58/collision/link_3.stl"/>
@@ -259,5 +266,5 @@
       </inertial>
       <visual>
-        <origin xyz="0 0 0" rpy="3.14159 3.14159 0"/>
+        <origin xyz="0 0 0" rpy="0 0 ${radians(180)}"/>
         <geometry>
           <mesh filename="package://abb_irb120_support/meshes/irb120_3_58/visual/link_4.stl"/>
@@ -266,5 +273,5 @@
       </visual>
       <collision>
-        <origin xyz="0 0 0" rpy="3.14159 3.14159 0"/>
+        <origin xyz="0 0 0" rpy="0 0 ${radians(180)}"/>
         <geometry>
           <mesh filename="package://abb_irb120_support/meshes/irb120_3_58/collision/link_4.stl"/>
@@ -280,5 +287,5 @@
       </inertial>
       <visual>
-        <origin xyz="0 0 0" rpy="3.14159 3.14159 0"/>
+        <origin xyz="0 0 0" rpy="0 0 ${radians(180)}"/>
         <geometry>
           <mesh filename="package://abb_irb120_support/meshes/irb120_3_58/visual/link_5.stl"/>
@@ -287,5 +294,5 @@
       </visual>
       <collision>
-        <origin xyz="0 0 0" rpy="3.14159 3.14159 0"/>
+        <origin xyz="0 0 0" rpy="0 0 ${radians(180)}"/>
         <geometry>
           <mesh filename="package://abb_irb120_support/meshes/irb120_3_58/collision/link_5.stl"/>
@@ -301,5 +308,5 @@
       </inertial>
       <visual>
-        <origin xyz="0 0 0" rpy="0 3.14159 0"/>
+        <origin xyz="0 0 0" rpy="0 0 ${radians(180)}"/>
         <geometry>
           <mesh filename="package://abb_irb120_support/meshes/irb120_3_58/visual/link_6.stl"/>
@@ -308,5 +315,5 @@
       </visual>
       <collision>
-        <origin xyz="0 0 0" rpy="0 3.14159 0"/>
+        <origin xyz="0 0 0" rpy="0 0 ${radians(180)}"/>
         <geometry>
           <mesh filename="package://abb_irb120_support/meshes/irb120_3_58/collision/link_6.stl"/>
@@ -342,4 +349,11 @@
         <xacro:material_abb_white />
       </visual>
+      <collision>
+        <origin xyz="0 0 0" rpy="0 0 0"/>
+        <geometry>
+          <mesh filename="package://abb_irb120_support/meshes/irb120_3_58/visual/cube.stl" scale="0.000001 0.000001 0.000001"/>
+        </geometry>
+        <xacro:material_abb_white />
+      </collision>
     </link>
     <!-- Arm 1 Joints -->
@@ -398,5 +412,5 @@
       <child link="${prefix}link_1_m"/>
       <limit effort="0" lower="-2.87979" upper="2.87979" velocity="4.36332"/>
-      <axis xyz="0 0 1"/>
+      <axis xyz="0 0 -1"/>
       <dynamics damping="0.0" friction="0.0"/>
     </joint>
@@ -438,5 +452,5 @@
       <child link="${prefix}link_6_m"/>
       <limit effort="0" lower="-6.98132" upper="6.98132" velocity="7.33038"/>
-      <axis xyz="1 0 0"/>
+      <axis xyz="-1 0 0"/>
       <dynamics damping="0.0" friction="0.0"/>
     </joint>

Commit message: [FIX] fix srdf and axis of rotation in urdf so that motion in RViz matches motino on robots, TFs in TF tree are all oriented with the same convention

File: abb_irb120_support/urdf/dual_arm_macro.xacro (robot description, xacro)
@@ -412,5 +412,5 @@
       <child link="${prefix}link_1_m"/>
       <limit effort="0" lower="-2.87979" upper="2.87979" velocity="4.36332"/>
-      <axis xyz="0 0 -1"/>
+      <axis xyz="0 0 1"/>
       <dynamics damping="0.0" friction="0.0"/>
     </joint>
