Commit message: [FIX] fix all URDF, SRDF, and STL files for properly publishing pointer TFs

File: abb_irb120_support/urdf/dual_arm_pointer_macro.xacro (robot description, xacro)
@@ -326,30 +326,9 @@
       <inertial>
         <mass value="0.137"/>
-        <origin xyz="0 0 0" rpy="0 0 0"/>
-        <inertia ixx="0.001" ixy="0" ixz="0" iyy="0.001" iyz="0" izz="0.001"/>
-      </inertial>
-      <visual>
-        <origin xyz="0 0 0" rpy="0 3.14159265 -1.5708"/>
-        <geometry>
-          <mesh filename="package://abb_irb120_support/meshes/irb120_3_58/visual/ABB_pointer.stl" scale="0.001 0.001 0.001"/>
-        </geometry>
-        <xacro:material_abb_black />
-      </visual>
-      <collision>
-        <origin xyz="0 0 0" rpy="0 3.14159265 -1.5708"/>
-        <geometry>
-          <mesh filename="package://abb_irb120_support/meshes/irb120_3_58/collision/ABB_pointer.stl" scale="0.001 0.001 0.001"/>
-        </geometry>
-        <xacro:material_abb_yellow />
-      </collision>
-    </link>
-    <link name="${prefix}pointer_m">
-      <inertial>
-        <mass value="0.137"/>
         <origin xyz="-0.00706 -0.00017 -1.32E-06" rpy="0 0 0"/>
         <inertia ixx="0.001" ixy="0" ixz="0" iyy="0.001" iyz="0" izz="0.001"/>
       </inertial>
       <visual>
-        <origin xyz="0 0.035 0.03" rpy="3.14159265 0 -1.5708"/>
+        <origin xyz="0 0 0" rpy="0 0 0"/>
         <geometry>
           <mesh filename="package://abb_irb120_support/meshes/irb120_3_58/visual/ABB_pointer.stl" scale="0.001 0.001 0.001"/>
@@ -358,5 +337,26 @@
       </visual>
       <collision>
-        <origin xyz="0 0 0" rpy="3.14159265 0 -1.5708"/>
+        <origin xyz="0 0 0" rpy="0 0 0"/>
+        <geometry>
+          <mesh filename="package://abb_irb120_support/meshes/irb120_3_58/collision/ABB_pointer.stl" scale="0.001 0.001 0.001"/>
+        </geometry>
+        <xacro:material_abb_yellow />
+      </collision>
+    </link>
+    <link name="${prefix}pointer_m">
+      <inertial>
+        <mass value="0.137"/>
+        <origin xyz="0 0 0" rpy="0 0 0"/>
+        <inertia ixx="0.001" ixy="0" ixz="0" iyy="0.001" iyz="0" izz="0.001"/>
+      </inertial>
+      <visual>
+        <origin xyz="0 0 0" rpy="0 0 ${radians(180)}"/>
+        <geometry>
+          <mesh filename="package://abb_irb120_support/meshes/irb120_3_58/visual/ABB_pointer.stl" scale="0.001 0.001 0.001"/>
+        </geometry>
+        <xacro:material_abb_black />
+      </visual>
+      <collision>
+        <origin xyz="0 0 0" rpy="0 0 ${radians(180)}"/>
         <geometry>
           <mesh filename="package://abb_irb120_support/meshes/irb120_3_58/collision/ABB_pointer.stl" scale="0.001 0.001 0.001"/>
@@ -464,13 +464,13 @@
     </joint>
     <!-- Pointer Joints -->
-    <joint name="${prefix}pointer_joint" type="fixed">
-      <origin rpy="0 0 0" xyz="0 -0.035 0.03"/>
-      <parent link="${prefix}link_6"/>
-      <child link="${prefix}pointer"/>
-    </joint>
     <joint name="${prefix}pointer_joint_m" type="fixed">
       <origin rpy="0 0 0" xyz="0 0 0"/>
       <parent link="${prefix}link_6_m"/>
       <child link="${prefix}pointer_m"/>
+    </joint>
+    <joint name="${prefix}pointer_joint" type="fixed">
+      <origin rpy="0 0 0" xyz="0 0 0"/>
+      <parent link="${prefix}link_6"/>
+      <child link="${prefix}pointer"/>
     </joint>
     <!-- World Joints -->

Commit message: [MODIFY] verfied robot-robot calibration and updated the parameters in URDF

File: abb_irb120_support/urdf/dual_arm_pointer_macro.xacro (robot description, xacro)
@@ -476,10 +476,10 @@
     <!-- World Joints -->
     <joint name="${prefix}world-base_link" type="fixed">
-      <origin xyz="-0.551 0 0" rpy="0 0 0"/>
+      <origin xyz="-0.548 0.0045 0" rpy="0 0 0"/>
       <parent link="${prefix}world"/>
       <child link="${prefix}base_link"/>
     </joint>
     <joint name="${prefix}world-base_link_m" type="fixed">
-      <origin xyz="0.551 0 0" rpy="0 0 0"/>
+      <origin xyz="0.548 -0.0045 0" rpy="0 0 0"/>
       <parent link="${prefix}world"/>
       <child link="${prefix}base_link_m"/>

Commit message: [FIX] urdf and srdf; pointer modifications

File: abb_irb120_support/urdf/dual_arm_pointer_macro.xacro (robot description, xacro)
@@ -474,12 +474,23 @@
       <child link="${prefix}pointer"/>
     </joint>
+    <!-- Pointer Tip Joints -->
+    <joint name="${prefix}pointer_joint_tip_m" type="fixed">
+      <origin rpy="0 0 0" xyz="0.03 0 -0.06"/>
+      <parent link="${prefix}pointer_m"/>
+      <child link="${prefix}pointer_tip_m"/>
+    </joint>
+    <joint name="${prefix}pointer_joint_tip" type="fixed">
+      <origin rpy="0 0 0" xyz="0.03 0 -0.06"/>
+      <parent link="${prefix}pointer"/>
+      <child link="${prefix}pointer_tip"/>
+    </joint>
     <!-- World Joints -->
     <joint name="${prefix}world-base_link" type="fixed">
-      <origin xyz="-0.548 0.0045 0" rpy="0 0 0"/>
+      <origin xyz="-0.551 -0.004 0" rpy="0 0 0"/>
       <parent link="${prefix}world"/>
       <child link="${prefix}base_link"/>
     </joint>
     <joint name="${prefix}world-base_link_m" type="fixed">
-      <origin xyz="0.548 -0.0045 0" rpy="0 0 0"/>
+      <origin xyz="0.551 0.004 0" rpy="0 0 0"/>
       <parent link="${prefix}world"/>
       <child link="${prefix}base_link_m"/>

Commit message: [VERIFY] moving world frame; touch test method

File: abb_irb120_support/urdf/dual_arm_pointer_macro.xacro (robot description, xacro)
@@ -332,5 +332,5 @@
         <origin xyz="0 0 0" rpy="0 0 0"/>
         <geometry>
-          <mesh filename="package://abb_irb120_support/meshes/irb120_3_58/visual/ABB_pointer.stl" scale="0.001 0.001 0.001"/>
+          <mesh filename="package://abb_irb120_support/meshes/irb120_3_58/visual/pointer_tip_frame.stl" scale="0.001 0.001 0.001"/>
         </geometry>
         <xacro:material_abb_black />
@@ -339,5 +339,5 @@
         <origin xyz="0 0 0" rpy="0 0 0"/>
         <geometry>
-          <mesh filename="package://abb_irb120_support/meshes/irb120_3_58/collision/ABB_pointer.stl" scale="0.001 0.001 0.001"/>
+          <mesh filename="package://abb_irb120_support/meshes/irb120_3_58/collision/pointer_tip_frame.stl" scale="0.001 0.001 0.001"/>
         </geometry>
         <xacro:material_abb_yellow />
@@ -353,5 +353,5 @@
         <origin xyz="0 0 0" rpy="0 0 ${radians(180)}"/>
         <geometry>
-          <mesh filename="package://abb_irb120_support/meshes/irb120_3_58/visual/ABB_pointer.stl" scale="0.001 0.001 0.001"/>
+          <mesh filename="package://abb_irb120_support/meshes/irb120_3_58/visual/pointer_tip_frame.stl" scale="0.001 0.001 0.001"/>
         </geometry>
         <xacro:material_abb_black />
@@ -360,5 +360,5 @@
         <origin xyz="0 0 0" rpy="0 0 ${radians(180)}"/>
         <geometry>
-          <mesh filename="package://abb_irb120_support/meshes/irb120_3_58/collision/ABB_pointer.stl" scale="0.001 0.001 0.001"/>
+          <mesh filename="package://abb_irb120_support/meshes/irb120_3_58/collision/pointer_tip_frame.stl" scale="0.001 0.001 0.001"/>
         </geometry>
         <xacro:material_abb_yellow />
@@ -465,32 +465,21 @@
     <!-- Pointer Joints -->
     <joint name="${prefix}pointer_joint_m" type="fixed">
-      <origin rpy="0 0 0" xyz="0 0 0"/>
+      <origin rpy="0 0 0" xyz="-0.03 0 -0.063"/>
       <parent link="${prefix}link_6_m"/>
       <child link="${prefix}pointer_m"/>
     </joint>
     <joint name="${prefix}pointer_joint" type="fixed">
-      <origin rpy="0 0 0" xyz="0 0 0"/>
+      <origin rpy="0 0 0" xyz="0.03 0 -0.063"/>
       <parent link="${prefix}link_6"/>
       <child link="${prefix}pointer"/>
     </joint>
-    <!-- Pointer Tip Joints -->
-    <joint name="${prefix}pointer_joint_tip_m" type="fixed">
-      <origin rpy="0 0 0" xyz="0.03 0 -0.06"/>
-      <parent link="${prefix}pointer_m"/>
-      <child link="${prefix}pointer_tip_m"/>
-    </joint>
-    <joint name="${prefix}pointer_joint_tip" type="fixed">
-      <origin rpy="0 0 0" xyz="0.03 0 -0.06"/>
-      <parent link="${prefix}pointer"/>
-      <child link="${prefix}pointer_tip"/>
-    </joint>
     <!-- World Joints -->
     <joint name="${prefix}world-base_link" type="fixed">
-      <origin xyz="-0.551 -0.004 0" rpy="0 0 0"/>
+      <origin xyz="-0.5455 -0.004 0" rpy="0 0 0"/>
       <parent link="${prefix}world"/>
       <child link="${prefix}base_link"/>
     </joint>
     <joint name="${prefix}world-base_link_m" type="fixed">
-      <origin xyz="0.551 0.004 0" rpy="0 0 0"/>
+      <origin xyz="0.5455 0.004 0" rpy="0 0 0"/>
       <parent link="${prefix}world"/>
       <child link="${prefix}base_link_m"/>
