Commit message: WORKING! - abb_pose_control node

File: abb_irb120_support/urdf/dual_arm_macro_pointer.xacro (robot description, xacro)
@@ -476,10 +476,10 @@
     <!-- World Joints -->
     <joint name="${prefix}world-base_link" type="fixed">
-      <origin xyz="-0.551 0 0" rpy="0 0 0"/>
+      <origin xyz="-0.556 0 0" rpy="0 0 0"/>
       <parent link="${prefix}world"/>
       <child link="${prefix}base_link"/>
     </joint>
     <joint name="${prefix}world-base_link_m" type="fixed">
-      <origin xyz="0.551 0 0" rpy="0 0 0"/>
+      <origin xyz="0.556 0 0" rpy="0 0 0"/>
       <parent link="${prefix}world"/>
       <child link="${prefix}base_link_m"/>

Commit message: [UPDATE] streamlining the process

File: abb_irb120_support/urdf/dual_arm_macro_pointer.xacro (robot description, xacro)
@@ -13,5 +13,5 @@
     <link name="${prefix}world">
       <visual>
-        <origin xyz="0 0 0" rpy="0 0 0"/>
+        <origin xyz="0 0 0.01" rpy="0 0 0"/>
         <geometry>
           <mesh filename="package://abb_irb120_support/meshes/irb120_3_58/visual/ground_plane.stl" scale="0.001 0.001 0.001"/>
@@ -20,5 +20,5 @@
       </visual>
       <collision>
-        <origin xyz="0 0 0" rpy="0 0 0"/>
+        <origin xyz="0 0 0.01" rpy="0 0 0"/>
         <geometry>
           <mesh filename="package://abb_irb120_support/meshes/irb120_3_58/collision/ground_plane.stl" scale="0.001 0.001 0.001"/>
@@ -476,10 +476,10 @@
     <!-- World Joints -->
     <joint name="${prefix}world-base_link" type="fixed">
-      <origin xyz="-0.556 0 0" rpy="0 0 0"/>
+      <origin xyz="-0.552 0 0.01" rpy="0 0 0"/>
       <parent link="${prefix}world"/>
       <child link="${prefix}base_link"/>
     </joint>
     <joint name="${prefix}world-base_link_m" type="fixed">
-      <origin xyz="0.556 0 0" rpy="0 0 0"/>
+      <origin xyz="0.552 0 0.01" rpy="0 0 0"/>
       <parent link="${prefix}world"/>
       <child link="${prefix}base_link_m"/>

File: abb_irb120_support/urdf/dual_arm_pointer_macro.xacro (robot description, xacro)
@@ -476,10 +476,10 @@
     <!-- World Joints -->
     <joint name="${prefix}world-base_link" type="fixed">
-      <origin xyz="-0.5455 -0.004 0" rpy="0 0 0"/>
+      <origin xyz="-0.5465 -0.004 0" rpy="0 0 0"/>
       <parent link="${prefix}world"/>
       <child link="${prefix}base_link"/>
     </joint>
     <joint name="${prefix}world-base_link_m" type="fixed">
-      <origin xyz="0.5455 0.004 0" rpy="0 0 0"/>
+      <origin xyz="0.5465 0.004 0" rpy="0 0 0"/>
       <parent link="${prefix}world"/>
       <child link="${prefix}base_link_m"/>
