Commit message: [UPDATE] changed the world frame location as per extrinsic calibration done in Sep. 2023

File: abb_irb120_support/urdf/dual_arm_gripper_macro.xacro (robot description, xacro)
@@ -474,10 +474,10 @@
     <!-- World Joints -->
     <joint name="${prefix}world-base_link" type="fixed">
-      <origin xyz="-0.545 0 0" rpy="0 0 0"/>
+      <origin xyz="-0.551 0 0" rpy="0 0 0"/>
       <parent link="${prefix}world"/>
       <child link="${prefix}base_link"/>
     </joint>
     <joint name="${prefix}world-base_link_m" type="fixed">
-      <origin xyz="0.545 0 0" rpy="0 0 0"/>
+      <origin xyz="0.551 0 0" rpy="0 0 0"/>
       <parent link="${prefix}world"/>
       <child link="${prefix}base_link_m"/>

File: abb_irb120_support/urdf/dual_arm_macro_pointer.xacro (robot description, xacro)
@@ -476,10 +476,10 @@
     <!-- World Joints -->
     <joint name="${prefix}world-base_link" type="fixed">
-      <origin xyz="-0.545 0 0" rpy="0 0 0"/>
+      <origin xyz="-0.551 0 0" rpy="0 0 0"/>
       <parent link="${prefix}world"/>
       <child link="${prefix}base_link"/>
     </joint>
     <joint name="${prefix}world-base_link_m" type="fixed">
-      <origin xyz="0.545 0 0" rpy="0 0 0"/>
+      <origin xyz="0.551 0 0" rpy="0 0 0"/>
       <parent link="${prefix}world"/>
       <child link="${prefix}base_link_m"/>

File: abb_irb120_support/urdf/dual_arm_pointer_macro.xacro (robot description, xacro)
@@ -476,10 +476,10 @@
     <!-- World Joints -->
     <joint name="${prefix}world-base_link" type="fixed">
-      <origin xyz="-0.545 0 0" rpy="0 0 0"/>
+      <origin xyz="-0.551 0 0" rpy="0 0 0"/>
       <parent link="${prefix}world"/>
       <child link="${prefix}base_link"/>
     </joint>
     <joint name="${prefix}world-base_link_m" type="fixed">
-      <origin xyz="0.545 0 0" rpy="0 0 0"/>
+      <origin xyz="0.551 0 0" rpy="0 0 0"/>
       <parent link="${prefix}world"/>
       <child link="${prefix}base_link_m"/>

Commit message: [FIX] update abb_joint_control with argparse for two sets of desired initial joint angle configs, update urdf tcp orientation for correct grasp alignment

File: abb_irb120_support/urdf/dual_arm_gripper_macro.xacro (robot description, xacro)
@@ -462,11 +462,10 @@
     </joint>
     <joint name="${prefix}gripper_base_joint_m" type="fixed">
-      <origin rpy="0 0 0" xyz="-0.1277 0 0"/>
+      <origin rpy="0 ${radians(90)} 0" xyz="-0.1277 0 0"/>
       <parent link="${prefix}gripper_m"/>
       <child link="${prefix}gripper_base_m"/>
     </joint>
     <joint name="${prefix}gripper_tcp_joint_m" type="fixed">
-      <!-- <origin rpy="0 0 0" xyz="-0.172 -0.0316545 0.0482436"/> -->
-      <origin rpy="${radians(-20)} 0 0" xyz="-0.045283 0 0"/>
+      <origin rpy="0 0 ${radians(-20)}" xyz="0 0 -0.045283"/>
       <parent link="${prefix}gripper_base_m"/>
       <child link="${prefix}gripper_tcp_m"/>

Commit message: [UPDATE] update urdf files with a collision cube for the d435 camera, update rviz files

File: abb_irb120_support/urdf/dual_arm_gripper_macro.xacro (robot description, xacro)
@@ -357,4 +357,20 @@
       </collision>
     </link>
+    <link name="${prefix}cube">
+      <visual>
+        <origin xyz="0.02 0 0" rpy="0 0 0"/>
+        <geometry>
+          <mesh filename="package://abb_irb120_support/meshes/irb120_3_58/visual/cube.stl" scale="0.0015 0.003 0.002"/>
+        </geometry>
+        <xacro:material_abb_white />
+      </visual>
+      <collision>
+        <origin xyz="0.02 0 0" rpy="0 0 0"/>
+        <geometry>
+          <mesh filename="package://abb_irb120_support/meshes/irb120_3_58/visual/cube.stl" scale="0.0015 0.003 0.002"/>
+        </geometry>
+        <xacro:material_abb_white />
+      </collision>
+    </link>
     <!-- Arm 1 Joints -->
     <joint name="${prefix}joint_2" type="revolute">
@@ -455,5 +471,5 @@
       <dynamics damping="0.0" friction="0.0"/>
     </joint>
-    <!-- Gripper Joints -->
+    <!-- End Effector Joints Joints -->
     <joint name="${prefix}gripper_joint_m" type="fixed">
       <origin rpy="0 0 0" xyz="0 0 0"/>
@@ -470,4 +486,9 @@
       <parent link="${prefix}gripper_base_m"/>
       <child link="${prefix}gripper_tcp_m"/>
+    </joint>
+    <joint name="${prefix}camera_collision_joint" type="fixed">
+      <origin rpy="0 0 0" xyz="0 0 0"/>
+      <parent link="${prefix}link_6"/>
+      <child link="${prefix}cube"/>
     </joint>
     <!-- World Joints -->

Commit message: [PREP] preparing to merge with Raghav's development of abb_dual_arm

File: abb_irb120_support/urdf/dual_arm_gripper_macro.xacro (robot description, xacro)
@@ -359,14 +359,14 @@
     <link name="${prefix}cube">
       <visual>
-        <origin xyz="0.02 0 0" rpy="0 0 0"/>
-        <geometry>
-          <mesh filename="package://abb_irb120_support/meshes/irb120_3_58/visual/cube.stl" scale="0.0015 0.003 0.002"/>
+        <origin xyz="0 0 0" rpy="0 0 0"/>
+        <geometry>
+          <mesh filename="package://abb_irb120_support/meshes/irb120_3_58/visual/cube.stl" scale="0.002 0.003 0.003"/>
         </geometry>
         <xacro:material_abb_white />
       </visual>
       <collision>
-        <origin xyz="0.02 0 0" rpy="0 0 0"/>
-        <geometry>
-          <mesh filename="package://abb_irb120_support/meshes/irb120_3_58/visual/cube.stl" scale="0.0015 0.003 0.002"/>
+        <origin xyz="0 0 0" rpy="0 0 0"/>
+        <geometry>
+          <mesh filename="package://abb_irb120_support/meshes/irb120_3_58/visual/cube.stl" scale="0.002 0.003 0.003"/>
         </geometry>
         <xacro:material_abb_white />
@@ -483,10 +483,10 @@
     </joint>
     <joint name="${prefix}gripper_tcp_joint_m" type="fixed">
-      <origin rpy="0 0 ${radians(-20)}" xyz="0 0 -0.045283"/>
+      <origin rpy="0 0 ${radians(-22.5)}" xyz="0 0 -0.0456"/>
       <parent link="${prefix}gripper_base_m"/>
       <child link="${prefix}gripper_tcp_m"/>
     </joint>
     <joint name="${prefix}camera_collision_joint" type="fixed">
-      <origin rpy="0 0 0" xyz="0 0 0"/>
+      <origin rpy="0 0 0" xyz="0.035 0 0"/>
       <parent link="${prefix}link_6"/>
       <child link="${prefix}cube"/>

Commit message: [RM, CAL] update arm-arm tf from calibration, rm two unused/redundant files

File: abb_irb120_support/urdf/dual_arm_gripper_macro.xacro (robot description, xacro)
@@ -494,10 +494,10 @@
     <!-- World Joints -->
     <joint name="${prefix}world-base_link" type="fixed">
-      <origin xyz="-0.545 0 0" rpy="0 0 0"/>
+      <origin xyz="-0.551 0 0.01" rpy="0 0 0"/>
       <parent link="${prefix}world"/>
       <child link="${prefix}base_link"/>
     </joint>
     <joint name="${prefix}world-base_link_m" type="fixed">
-      <origin xyz="0.545 0 0" rpy="0 0 0"/>
+      <origin xyz="0.551 0 0.01" rpy="0 0 0"/>
       <parent link="${prefix}world"/>
       <child link="${prefix}base_link_m"/>

Commit message: [CI, CAL] update CI to rm ubuntu 18.04 from os matrix (no longer supported by github actions) and update dual_arm_gripper urdf with new arm-world calibration

File: abb_irb120_support/urdf/dual_arm_gripper_macro.xacro (robot description, xacro)
@@ -494,10 +494,10 @@
     <!-- World Joints -->
     <joint name="${prefix}world-base_link" type="fixed">
-      <origin xyz="-0.551 0 0.01" rpy="0 0 0"/>
+      <origin xyz="-0.552 0 0.01" rpy="0 0 0"/>
       <parent link="${prefix}world"/>
       <child link="${prefix}base_link"/>
     </joint>
     <joint name="${prefix}world-base_link_m" type="fixed">
-      <origin xyz="0.551 0 0.01" rpy="0 0 0"/>
+      <origin xyz="0.552 0 0.01" rpy="0 0 0"/>
       <parent link="${prefix}world"/>
       <child link="${prefix}base_link_m"/>

Commit message: [VIZ, DEVEL] update visualizations (re-scale/size .stl files, change mesh color, add record.rviz) and add r1_twist func in abb_track_point

File: abb_irb120_support/urdf/dual_arm_gripper_macro.xacro (robot description, xacro)
@@ -15,12 +15,12 @@
         <origin xyz="0 0 0" rpy="0 0 0"/>
         <geometry>
-          <mesh filename="package://abb_irb120_support/meshes/irb120_3_58/visual/ground_plane.stl" scale="0.001 0.001 0.001"/>
-        </geometry>
-        <xacro:material_abb_white />
-      </visual>
-      <collision>
-        <origin xyz="0 0 0" rpy="0 0 0"/>
-        <geometry>
-          <mesh filename="package://abb_irb120_support/meshes/irb120_3_58/collision/ground_plane.stl" scale="0.001 0.001 0.001"/>
+          <mesh filename="package://abb_irb120_support/meshes/irb120_3_58/visual/ground_plane.stl"/>
+        </geometry>
+        <xacro:material_abb_white />
+      </visual>
+      <collision>
+        <origin xyz="0 0 0" rpy="0 0 0"/>
+        <geometry>
+          <mesh filename="package://abb_irb120_support/meshes/irb120_3_58/collision/ground_plane.stl"/>
         </geometry>
       </collision>
@@ -38,5 +38,5 @@
           <mesh filename="package://abb_irb120_support/meshes/irb120_3_58/visual/base_link.stl"/>
         </geometry>
-        <xacro:material_abb_orange />
+        <xacro:material_abb_white />
       </visual>
       <collision>
@@ -59,5 +59,5 @@
           <mesh filename="package://abb_irb120_support/meshes/irb120_3_58/visual/link_1.stl"/>
         </geometry>
-        <xacro:material_abb_orange />
+        <xacro:material_abb_white />
       </visual>
       <collision>
@@ -80,5 +80,5 @@
           <mesh filename="package://abb_irb120_support/meshes/irb120_3_58/visual/link_2.stl"/>
         </geometry>
-        <xacro:material_abb_orange />
+        <xacro:material_abb_white />
       </visual>
       <collision>
@@ -101,5 +101,5 @@
           <mesh filename="package://abb_irb120_support/meshes/irb120_3_58/visual/link_3.stl"/>
         </geometry>
-        <xacro:material_abb_orange />
+        <xacro:material_abb_white />
       </visual>
       <collision>
@@ -122,5 +122,5 @@
           <mesh filename="package://abb_irb120_support/meshes/irb120_3_58/visual/link_4.stl"/>
         </geometry>
-        <xacro:material_abb_orange />
+        <xacro:material_abb_white />
       </visual>
       <collision>
@@ -143,5 +143,5 @@
           <mesh filename="package://abb_irb120_support/meshes/irb120_3_58/visual/link_5.stl"/>
         </geometry>
-        <xacro:material_abb_orange />
+        <xacro:material_abb_white />
       </visual>
       <collision>
@@ -186,5 +186,5 @@
           <mesh filename="package://abb_irb120_support/meshes/irb120_3_58/visual/base_link.stl"/>
         </geometry>
-        <xacro:material_abb_orange />
+        <xacro:material_abb_white />
       </visual>
       <collision>
@@ -207,5 +207,5 @@
           <mesh filename="package://abb_irb120_support/meshes/irb120_3_58/visual/link_1.stl"/>
         </geometry>
-        <xacro:material_abb_orange />
+        <xacro:material_abb_white />
       </visual>
       <collision>
@@ -228,5 +228,5 @@
           <mesh filename="package://abb_irb120_support/meshes/irb120_3_58/visual/link_2.stl"/>
         </geometry>
-        <xacro:material_abb_orange />
+        <xacro:material_abb_white />
       </visual>
       <collision>
@@ -249,5 +249,5 @@
           <mesh filename="package://abb_irb120_support/meshes/irb120_3_58/visual/link_3.stl"/>
         </geometry>
-        <xacro:material_abb_orange />
+        <xacro:material_abb_white />
       </visual>
       <collision>
@@ -270,5 +270,5 @@
           <mesh filename="package://abb_irb120_support/meshes/irb120_3_58/visual/link_4.stl"/>
         </geometry>
-        <xacro:material_abb_orange />
+        <xacro:material_abb_white />
       </visual>
       <collision>
@@ -291,5 +291,5 @@
           <mesh filename="package://abb_irb120_support/meshes/irb120_3_58/visual/link_5.stl"/>
         </geometry>
-        <xacro:material_abb_orange />
+        <xacro:material_abb_white />
       </visual>
       <collision>
@@ -327,12 +327,12 @@
         <origin xyz="0 0 0" rpy="0 0 0"/>
         <geometry>
-          <mesh filename="package://abb_irb120_support/meshes/irb120_3_58/visual/gripper_assembly.stl" scale="0.001 0.001 0.001"/>
-        </geometry>
-        <xacro:material_abb_white />
-      </visual>
-      <collision>
-        <origin xyz="0 0 0" rpy="0 0 0"/>
-        <geometry>
-          <mesh filename="package://abb_irb120_support/meshes/irb120_3_58/collision/gripper_collision_cube.stl" scale="0.001 0.001 0.001"/>
+          <mesh filename="package://abb_irb120_support/meshes/irb120_3_58/visual/gripper_assembly.stl"/>
+        </geometry>
+        <xacro:material_abb_white />
+      </visual>
+      <collision>
+        <origin xyz="0 0 0" rpy="0 0 0"/>
+        <geometry>
+          <mesh filename="package://abb_irb120_support/meshes/irb120_3_58/collision/gripper_collision_cube.stl"/>
         </geometry>
       </collision>

File: abb_irb120_support/urdf/dual_arm_macro_pointer.xacro (robot description, xacro)
@@ -15,5 +15,5 @@
         <origin xyz="0 0 0.01" rpy="0 0 0"/>
         <geometry>
-          <mesh filename="package://abb_irb120_support/meshes/irb120_3_58/visual/ground_plane.stl" scale="0.001 0.001 0.001"/>
+          <mesh filename="package://abb_irb120_support/meshes/irb120_3_58/visual/ground_plane.stl"/>
         </geometry>
         <xacro:material_abb_white />
@@ -22,5 +22,5 @@
         <origin xyz="0 0 0.01" rpy="0 0 0"/>
         <geometry>
-          <mesh filename="package://abb_irb120_support/meshes/irb120_3_58/collision/ground_plane.stl" scale="0.001 0.001 0.001"/>
+          <mesh filename="package://abb_irb120_support/meshes/irb120_3_58/collision/ground_plane.stl"/>
         </geometry>
       </collision>
@@ -38,5 +38,5 @@
           <mesh filename="package://abb_irb120_support/meshes/irb120_3_58/visual/base_link.stl"/>
         </geometry>
-        <xacro:material_abb_orange />
+        <xacro:material_abb_white />
       </visual>
       <collision>
@@ -59,5 +59,5 @@
           <mesh filename="package://abb_irb120_support/meshes/irb120_3_58/visual/link_1.stl"/>
         </geometry>
-        <xacro:material_abb_orange />
+        <xacro:material_abb_white />
       </visual>
       <collision>
@@ -80,5 +80,5 @@
           <mesh filename="package://abb_irb120_support/meshes/irb120_3_58/visual/link_2.stl"/>
         </geometry>
-        <xacro:material_abb_orange />
+        <xacro:material_abb_white />
       </visual>
       <collision>
@@ -101,5 +101,5 @@
           <mesh filename="package://abb_irb120_support/meshes/irb120_3_58/visual/link_3.stl"/>
         </geometry>
-        <xacro:material_abb_orange />
+        <xacro:material_abb_white />
       </visual>
       <collision>
@@ -122,5 +122,5 @@
           <mesh filename="package://abb_irb120_support/meshes/irb120_3_58/visual/link_4.stl"/>
         </geometry>
-        <xacro:material_abb_orange />
+        <xacro:material_abb_white />
       </visual>
       <collision>
@@ -143,5 +143,5 @@
           <mesh filename="package://abb_irb120_support/meshes/irb120_3_58/visual/link_5.stl"/>
         </geometry>
-        <xacro:material_abb_orange />
+        <xacro:material_abb_white />
       </visual>
       <collision>
@@ -186,5 +186,5 @@
           <mesh filename="package://abb_irb120_support/meshes/irb120_3_58/visual/base_link.stl"/>
         </geometry>
-        <xacro:material_abb_orange />
+        <xacro:material_abb_white />
       </visual>
       <collision>
@@ -207,5 +207,5 @@
           <mesh filename="package://abb_irb120_support/meshes/irb120_3_58/visual/link_1.stl"/>
         </geometry>
-        <xacro:material_abb_orange />
+        <xacro:material_abb_white />
       </visual>
       <collision>
@@ -228,5 +228,5 @@
           <mesh filename="package://abb_irb120_support/meshes/irb120_3_58/visual/link_2.stl"/>
         </geometry>
-        <xacro:material_abb_orange />
+        <xacro:material_abb_white />
       </visual>
       <collision>
@@ -249,5 +249,5 @@
           <mesh filename="package://abb_irb120_support/meshes/irb120_3_58/visual/link_3.stl"/>
         </geometry>
-        <xacro:material_abb_orange />
+        <xacro:material_abb_white />
       </visual>
       <collision>
@@ -270,5 +270,5 @@
           <mesh filename="package://abb_irb120_support/meshes/irb120_3_58/visual/link_4.stl"/>
         </geometry>
-        <xacro:material_abb_orange />
+        <xacro:material_abb_white />
       </visual>
       <collision>
@@ -291,5 +291,5 @@
           <mesh filename="package://abb_irb120_support/meshes/irb120_3_58/visual/link_5.stl"/>
         </geometry>
-        <xacro:material_abb_orange />
+        <xacro:material_abb_white />
       </visual>
       <collision>

File: abb_irb120_support/urdf/dual_arm_pointer_macro.xacro (robot description, xacro)
@@ -15,12 +15,12 @@
         <origin xyz="0 0 0" rpy="0 0 0"/>
         <geometry>
-          <mesh filename="package://abb_irb120_support/meshes/irb120_3_58/visual/ground_plane.stl" scale="0.001 0.001 0.001"/>
-        </geometry>
-        <xacro:material_abb_white />
-      </visual>
-      <collision>
-        <origin xyz="0 0 0" rpy="0 0 0"/>
-        <geometry>
-          <mesh filename="package://abb_irb120_support/meshes/irb120_3_58/collision/ground_plane.stl" scale="0.001 0.001 0.001"/>
+          <mesh filename="package://abb_irb120_support/meshes/irb120_3_58/visual/ground_plane.stl"/>
+        </geometry>
+        <xacro:material_abb_white />
+      </visual>
+      <collision>
+        <origin xyz="0 0 0" rpy="0 0 0"/>
+        <geometry>
+          <mesh filename="package://abb_irb120_support/meshes/irb120_3_58/collision/ground_plane.stl"/>
         </geometry>
       </collision>
@@ -38,5 +38,5 @@
           <mesh filename="package://abb_irb120_support/meshes/irb120_3_58/visual/base_link.stl"/>
         </geometry>
-        <xacro:material_abb_orange />
+        <xacro:material_abb_white />
       </visual>
       <collision>
@@ -59,5 +59,5 @@
           <mesh filename="package://abb_irb120_support/meshes/irb120_3_58/visual/link_1.stl"/>
         </geometry>
-        <xacro:material_abb_orange />
+        <xacro:material_abb_white />
       </visual>
       <collision>
@@ -80,5 +80,5 @@
           <mesh filename="package://abb_irb120_support/meshes/irb120_3_58/visual/link_2.stl"/>
         </geometry>
-        <xacro:material_abb_orange />
+        <xacro:material_abb_white />
       </visual>
       <collision>
@@ -101,5 +101,5 @@
           <mesh filename="package://abb_irb120_support/meshes/irb120_3_58/visual/link_3.stl"/>
         </geometry>
-        <xacro:material_abb_orange />
+        <xacro:material_abb_white />
       </visual>
       <collision>
@@ -122,5 +122,5 @@
           <mesh filename="package://abb_irb120_support/meshes/irb120_3_58/visual/link_4.stl"/>
         </geometry>
-        <xacro:material_abb_orange />
+        <xacro:material_abb_white />
       </visual>
       <collision>
@@ -143,5 +143,5 @@
           <mesh filename="package://abb_irb120_support/meshes/irb120_3_58/visual/link_5.stl"/>
         </geometry>
-        <xacro:material_abb_orange />
+        <xacro:material_abb_white />
       </visual>
       <collision>
@@ -186,5 +186,5 @@
           <mesh filename="package://abb_irb120_support/meshes/irb120_3_58/visual/base_link.stl"/>
         </geometry>
-        <xacro:material_abb_orange />
+        <xacro:material_abb_white />
       </visual>
       <collision>
@@ -207,5 +207,5 @@
           <mesh filename="package://abb_irb120_support/meshes/irb120_3_58/visual/link_1.stl"/>
         </geometry>
-        <xacro:material_abb_orange />
+        <xacro:material_abb_white />
       </visual>
       <collision>
@@ -228,5 +228,5 @@
           <mesh filename="package://abb_irb120_support/meshes/irb120_3_58/visual/link_2.stl"/>
         </geometry>
-        <xacro:material_abb_orange />
+        <xacro:material_abb_white />
       </visual>
       <collision>
@@ -249,5 +249,5 @@
           <mesh filename="package://abb_irb120_support/meshes/irb120_3_58/visual/link_3.stl"/>
         </geometry>
-        <xacro:material_abb_orange />
+        <xacro:material_abb_white />
       </visual>
       <collision>
@@ -270,5 +270,5 @@
           <mesh filename="package://abb_irb120_support/meshes/irb120_3_58/visual/link_4.stl"/>
         </geometry>
-        <xacro:material_abb_orange />
+        <xacro:material_abb_white />
       </visual>
       <collision>
@@ -291,5 +291,5 @@
           <mesh filename="package://abb_irb120_support/meshes/irb120_3_58/visual/link_5.stl"/>
         </geometry>
-        <xacro:material_abb_orange />
+        <xacro:material_abb_white />
       </visual>
       <collision>

Commit message: [ADD] add camera .stl file to dual arm urdf

File: abb_irb120_support/urdf/dual_arm_gripper_macro.xacro (robot description, xacro)
@@ -357,9 +357,9 @@
       </collision>
     </link>
-    <link name="${prefix}cube">
-      <visual>
-        <origin xyz="0 0 0" rpy="0 0 0"/>
-        <geometry>
-          <mesh filename="package://abb_irb120_support/meshes/irb120_3_58/visual/cube.stl" scale="0.002 0.003 0.003"/>
+    <link name="${prefix}camera">
+      <visual>
+        <origin xyz="0 0 0" rpy="0 0 0"/>
+        <geometry>
+          <mesh filename="package://abb_irb120_support/meshes/irb120_3_58/visual/d415.stl"/>
         </geometry>
         <xacro:material_abb_white />
@@ -488,7 +488,7 @@
     </joint>
     <joint name="${prefix}camera_collision_joint" type="fixed">
-      <origin rpy="0 0 0" xyz="0.035 0 0"/>
+      <origin rpy="0 0 0" xyz="0.01801587 0.0156162 -0.03926776"/>
       <parent link="${prefix}link_6"/>
-      <child link="${prefix}cube"/>
+      <child link="${prefix}camera"/>
     </joint>
     <!-- World Joints -->

Commit message: [FIX] fix camera collision cube in collision with link_6 on mp in urdf, srdf, update viz

File: abb_irb120_support/urdf/dual_arm_gripper_macro.xacro (robot description, xacro)
@@ -368,5 +368,5 @@
         <origin xyz="0 0 0" rpy="0 0 0"/>
         <geometry>
-          <mesh filename="package://abb_irb120_support/meshes/irb120_3_58/visual/cube.stl" scale="0.002 0.003 0.003"/>
+          <mesh filename="package://abb_irb120_support/meshes/irb120_3_58/visual/cube.stl" scale="0.0012 0.0035 0.002"/>
         </geometry>
         <xacro:material_abb_white />

Commit message: [FIX] add positive y offset for mp_m_base_link to world - more accurate cal

File: abb_irb120_support/urdf/dual_arm_gripper_macro.xacro (robot description, xacro)
@@ -499,5 +499,5 @@
     </joint>
     <joint name="${prefix}world-base_link_m" type="fixed">
-      <origin xyz="0.552 0 0.01" rpy="0 0 0"/>
+      <origin xyz="0.552 0.02 0.01" rpy="0 0 0"/>
       <parent link="${prefix}world"/>
       <child link="${prefix}base_link_m"/>

Commit message: [MINOR] update record.rviz, set initial mp_m config with link_6_m rotated -90 degrees

File: abb_irb120_support/urdf/dual_arm_gripper_macro.xacro (robot description, xacro)
@@ -456,5 +456,5 @@
     </joint>
     <joint name="${prefix}joint_6_m" type="revolute">
-      <origin rpy="0 0 0" xyz="-0.302 0 0"/>
+      <origin rpy="0 ${radians(-90)} 0" xyz="-0.302 0 0"/>
       <parent link="${prefix}link_4_m"/>
       <child link="${prefix}link_5_m"/>
