Commit message: [ADD, FIX] add record_from_rosbag.rviz, used with knot.launch sim_pub:=true, and fixed a rotated gripper in urdf that resulted in bad bag playback

File: abb_irb120_support/urdf/dual_arm_gripper_macro.xacro (robot description, xacro)
@@ -456,5 +456,5 @@
     </joint>
     <joint name="${prefix}joint_6_m" type="revolute">
-      <origin rpy="0 ${radians(-90)} 0" xyz="-0.302 0 0"/>
+      <origin rpy="0 0 0" xyz="-0.302 0 0"/>
       <parent link="${prefix}link_4_m"/>
       <child link="${prefix}link_5_m"/>

Commit message: [ADD] add camera mount.stl mesh files and description to urdf

File: abb_irb120_support/urdf/dual_arm_gripper_macro.xacro (robot description, xacro)
@@ -373,4 +373,20 @@
       </collision>
     </link>
+    <link name="${prefix}camera_mount">
+      <visual>
+        <origin xyz="0 0 0" rpy="0 0 0"/>
+        <geometry>
+          <mesh filename="package://abb_irb120_support/meshes/irb120_3_58/visual/camera_mount.stl"/>
+        </geometry>
+        <xacro:material_abb_white />
+      </visual>
+      <collision>
+        <origin xyz="0 0 0" rpy="0 0 0"/>
+        <geometry>
+          <mesh filename="package://abb_irb120_support/meshes/irb120_3_58/visual/cube.stl" scale="0.0001 0.0003 0.0001"/>
+        </geometry>
+        <xacro:material_abb_white />
+      </collision>
+    </link>
     <!-- Arm 1 Joints -->
     <joint name="${prefix}joint_2" type="revolute">
@@ -456,5 +472,6 @@
     </joint>
     <joint name="${prefix}joint_6_m" type="revolute">
-      <origin rpy="0 ${radians(-90)} 0" xyz="-0.302 0 0"/>
+      <!-- <origin rpy="0 ${radians(-90)} 0" xyz="-0.302 0 0"/> -->
+      <origin rpy="0 0 0" xyz="-0.302 0 0"/>
       <parent link="${prefix}link_4_m"/>
       <child link="${prefix}link_5_m"/>
@@ -487,6 +504,11 @@
       <child link="${prefix}gripper_tcp_m"/>
     </joint>
+    <joint name="${prefix}camera_mount_joint" type="fixed">
+      <origin rpy="0 0 0" xyz="0 0 0"/>
+      <parent link="${prefix}link_6"/>
+      <child link="${prefix}camera_mount"/>
+    </joint>
     <joint name="${prefix}camera_collision_joint" type="fixed">
-      <origin rpy="0 0 0" xyz="0.01801587 0.0156162 -0.03926776"/>
+      <origin rpy="0 0 0" xyz="0.01 0 -0.0373"/>
       <parent link="${prefix}link_6"/>
       <child link="${prefix}camera"/>

Commit message: [UPDATE] update camera and camera mount collision origins and scales

File: abb_irb120_support/urdf/dual_arm_gripper_macro.xacro (robot description, xacro)
@@ -366,7 +366,7 @@
       </visual>
       <collision>
-        <origin xyz="0 0 0" rpy="0 0 0"/>
-        <geometry>
-          <mesh filename="package://abb_irb120_support/meshes/irb120_3_58/visual/cube.stl" scale="0.0012 0.0035 0.002"/>
+        <origin xyz="0.001 0 0.013" rpy="0 0 0"/>
+        <geometry>
+          <mesh filename="package://abb_irb120_support/meshes/irb120_3_58/visual/cube.stl" scale="0.0007 0.0035 0.001"/>
         </geometry>
         <xacro:material_abb_white />
@@ -384,5 +384,5 @@
         <origin xyz="0 0 0" rpy="0 0 0"/>
         <geometry>
-          <mesh filename="package://abb_irb120_support/meshes/irb120_3_58/visual/cube.stl" scale="0.0001 0.0003 0.0001"/>
+          <mesh filename="package://abb_irb120_support/meshes/irb120_3_58/visual/cube.stl" scale="0.000001 0.000001 0.000001"/>
         </geometry>
         <xacro:material_abb_white />

Commit message: [MAJOR] computing reachability (script, doc, config.json, image), update frames.pdf with camera and gripper, update rviz files, update links in urdf and srdf

File: abb_irb120_support/urdf/dual_arm_gripper_macro.xacro (robot description, xacro)
@@ -514,10 +514,10 @@
     </joint>
     <!-- World Joints -->
-    <joint name="${prefix}world-base_link" type="fixed">
+    <joint name="${prefix}world_joint" type="fixed">
       <origin xyz="-0.552 0 0.01" rpy="0 0 0"/>
       <parent link="${prefix}world"/>
       <child link="${prefix}base_link"/>
     </joint>
-    <joint name="${prefix}world-base_link_m" type="fixed">
+    <joint name="${prefix}world_joint_m" type="fixed">
       <origin xyz="0.552 0.02 0.01" rpy="0 0 0"/>
       <parent link="${prefix}world"/>

Commit message: [MINOR] minor changes to test computing cartesian path and address launch warnings

File: abb_irb120_support/urdf/dual_arm_gripper_macro.xacro (robot description, xacro)
@@ -472,5 +472,5 @@
     </joint>
     <joint name="${prefix}joint_6_m" type="revolute">
-      <origin rpy="0 ${radians(-90)} 0" xyz="-0.302 0 0"/>
+      <origin rpy="0 0 0" xyz="-0.302 0 0"/>
       <parent link="${prefix}link_4_m"/>
       <child link="${prefix}link_5_m"/>
@@ -492,4 +492,5 @@
       <parent link="${prefix}link_6_m"/>
       <child link="${prefix}gripper_m"/>
+      <limit effort="0" lower="0" upper="0" velocity="0"/>
     </joint>
     <joint name="${prefix}gripper_base_joint_m" type="fixed">
@@ -497,4 +498,5 @@
       <parent link="${prefix}gripper_m"/>
       <child link="${prefix}gripper_base_m"/>
+      <limit effort="0" lower="0" upper="0" velocity="0"/>
     </joint>
     <joint name="${prefix}gripper_tcp_joint_m" type="fixed">
@@ -502,4 +504,5 @@
       <parent link="${prefix}gripper_base_m"/>
       <child link="${prefix}gripper_tcp_m"/>
+      <limit effort="0" lower="0" upper="0" velocity="0"/>
     </joint>
     <joint name="${prefix}camera_mount_joint" type="fixed">
@@ -507,9 +510,11 @@
       <parent link="${prefix}link_6"/>
       <child link="${prefix}camera_mount"/>
+      <limit effort="0" lower="0" upper="0" velocity="0"/>
     </joint>
     <joint name="${prefix}camera_collision_joint" type="fixed">
       <origin rpy="0 0 0" xyz="0.01 0 -0.0373"/>
-      <parent link="${prefix}link_6"/>
+      <parent link="${prefix}camera_mount"/>
       <child link="${prefix}camera"/>
+      <limit effort="0" lower="0" upper="0" velocity="0"/>
     </joint>
     <!-- World Joints -->
@@ -518,4 +523,5 @@
       <parent link="${prefix}world"/>
       <child link="${prefix}base_link"/>
+      <limit effort="0" lower="0" upper="0" velocity="0"/>
     </joint>
     <joint name="${prefix}world_joint_m" type="fixed">
@@ -523,4 +529,5 @@
       <parent link="${prefix}world"/>
       <child link="${prefix}base_link_m"/>
+      <limit effort="0" lower="0" upper="0" velocity="0"/>
     </joint>
   </xacro:macro>
